Commit message: 2021-1-13

File: src/probot_description/urdf/probot_anno_with_gripper.xacro (robot description, xacro)
@@ -2,4 +2,6 @@
 <robot name="probot_anno" xmlns:xacro="http://ros.org/wiki/xacro">
   <xacro:property name="M_PI" value="3.1415926536"/>
+  <xacro:include filename="$(find probot_description)/urdf/materials.urdf.xacro" />
+  <xacro:include filename="$(find probot_description)/urdf/gripper.xacro" />
   <link name="base_footprint"/>
   <joint name="joint_0" type="fixed">
@@ -11,6 +13,6 @@
     <inertial>
       <origin xyz="-0.010934 0.23134 0.0051509" rpy="0 0 0" />
-      <mass value="19.574" />
-      <inertia ixx="0" ixy="0" ixz="0" iyy="0" iyz="0" izz="0" />
+      <mass value="0.01" />
+      <inertia ixx="1.0" ixy="0.0" ixz="0.0" iyy="1.0" iyz="0.0" izz="1.0" />
     </inertial>
     <visual>
@@ -33,6 +35,6 @@
     <inertial>
       <origin xyz="-0.010934 0.23134 0.0051509" rpy="0 0 0" />
-      <mass value="19.574" />
-      <inertia ixx="0" ixy="0" ixz="0" iyy="0" iyz="0" izz="0" />
+      <mass value="0.01" />
+      <inertia ixx="1.0" ixy="0.0" ixz="0.0" iyy="1.0" iyz="0.0" izz="1.0" />
     </inertial>
     <visual>
@@ -62,6 +64,6 @@
     <inertial>
       <origin xyz="-0.010934 0.23134 0.0051509" rpy="0 0 0" />
-      <mass value="19.574" />
-      <inertia ixx="0" ixy="0" ixz="0" iyy="0" iyz="0" izz="0" />
+      <mass value="0.001" />
+        <inertia ixx="1.0" ixy="0.0" ixz="0.0" iyy="1.0" iyz="0.0" izz="1.0" />
     </inertial>
     <visual>
@@ -91,6 +93,6 @@
     <inertial>
       <origin xyz="-0.010934 0.23134 0.0051509" rpy="0 0 0" />
-      <mass value="19.574" />
-      <inertia ixx="0" ixy="0" ixz="0" iyy="0" iyz="0" izz="0" />
+      <mass value="0.001" />
+        <inertia ixx="1.0" ixy="0.0" ixz="0.0" iyy="1.0" iyz="0.0" izz="1.0" />
     </inertial>
     <visual>
@@ -120,6 +122,6 @@
     <inertial>
       <origin xyz="-0.010934 0.23134 0.0051509" rpy="0 0 0" />
-      <mass value="19.574" />
-      <inertia ixx="0" ixy="0" ixz="0" iyy="0" iyz="0" izz="0" />
+      <mass value="0.00001" />
+      <inertia ixx="1.0" ixy="0.0" ixz="0.0" iyy="1.0" iyz="0.0" izz="1.0" />
     </inertial>
     <visual>
@@ -149,6 +151,6 @@
     <inertial>
       <origin xyz="-0.010934 0.23134 0.0051509" rpy="0 0 0" />
-      <mass value="19.574" />
-      <inertia ixx="0" ixy="0" ixz="0" iyy="0" iyz="0" izz="0" />
+      <mass value="0.00001" />
+      <inertia ixx="1.0" ixy="0.0" ixz="0.0" iyy="1.0" iyz="0.0" izz="1.0" />
     </inertial>
     <visual>
@@ -178,6 +180,6 @@
     <inertial>
       <origin xyz="-0.010934 0.23134 0.0051509" rpy="0 0 0" />
-      <mass value="19.574" />
-      <inertia ixx="0" ixy="0" ixz="0" iyy="0" iyz="0" izz="0" />
+      <mass value="0.00001" />
+      <inertia ixx="1.0" ixy="0.0" ixz="0.0" iyy="1.0" iyz="0.0" izz="1.0" />
     </inertial>
     <visual>
@@ -206,8 +208,10 @@
   <link name="tool0"/>
   <joint name="joint_tool0" type="fixed">
-    <origin xyz="0 -0.013 0" rpy="0 0 0" />
+    <origin xyz="0 -0.02 0" rpy="0 0 0" />
     <parent link="link_6" />
     <child link="tool0" />
   </joint>
+   <!-- Attach the right gripper -->
+   <gripper parent="tool0" color="Green" xyz="0 -0.015 0.01" rpy="0 0 ${-M_PI/2}"/>
   <!-- Transmissions for ROS Control -->
   <xacro:macro name="transmission_block" params="joint_name">
@@ -229,4 +233,6 @@
   <xacro:transmission_block joint_name="joint_5"/>
   <xacro:transmission_block joint_name="joint_6"/>
+  <xacro:transmission_block joint_name="gripper_finger_joint"/>
+  <xacro:include filename="$(find probot_description)/urdf/sensors/camera.urdf.xacro"/>
   <!-- ros_control plugin -->
   <gazebo>
